Commit message: 实现平地控制，但是机械臂控制重心部分还要调

File: source/excavator_ppo/excavator_ppo/robots/excavator_six_wheels/urdf/excavator_six_wheels.urdf (robot description, URDF)
Before this commit: robot excavator_six_wheels, 11 links, 10 joints
Links:
- link base_link: mass 1344.5600138 -> 1344.56
- link body_yaw_link: mass 15120.6382761 -> 6265.561
- link boom_pitch_link: mass 724.9528599 -> 724.9529
- link bucket_pitch_link: mass 643.2329046 -> 643.2329
- link forearm_pitch_link: mass 640.9527498 -> 640.9527
- link left_behind_wheel_link: mass 80.8643451 -> 80.86435
- link left_front_wheel_link: mass 80.8643451 -> 80.86435
- link left_wheel_link: mass 80.8643451 -> 80.86435
- link right_behind_wheel_link: mass 80.8643451 -> 80.86435
- link right_front_wheel_link: mass 80.8643451 -> 80.86435
- link right_wheel_link: mass 80.8643451 -> 80.86435
Joints:
- joint boom_pitch_joint: origin xyz=1.5882 0.039526 0.36333 rpy=-1.5708 0 0 -> xyz=1.5923 -0.0015397 0.36333 rpy=-1.5708 0 0
- joint bucket_pitch_joint: origin xyz=1.4765 -0.24997 0.29735 rpy=0 0 0 -> xyz=1.5061 -0.24997 0 rpy=0 0 0
- joint forearm_pitch_joint: origin xyz=1.4233 -2.0381 0.28664 rpy=0 0 0 -> xyz=1.4519 -2.0381 0 rpy=0 0 0
- joint left_behind_wheel_joint: origin xyz=-0.96819 1.1184 0 rpy=-1.5708 0 0 -> xyz=-0.96819 0.76843 0 rpy=-1.5708 0 0
- joint left_front_wheel_joint: origin xyz=0.90862 1.1184 0 rpy=-1.5708 0 0 -> xyz=0.90862 0.76843 0 rpy=-1.5708 0 0
- joint left_wheel_joint: origin xyz=-0.029784 1.1184 0 rpy=-1.5708 0 0 -> xyz=-0.029784 0.76843 0 rpy=-1.5708 0 0
- joint right_behind_wheel_joint: origin xyz=-0.96819 -1.1174 0 rpy=-1.5708 0 0 -> xyz=-0.96819 -0.76743 0 rpy=-1.5708 0 0
- joint right_front_wheel_joint: origin xyz=0.90862 -1.1179 0 rpy=-1.5708 0 0 -> xyz=0.90862 -0.76743 0 rpy=-1.5708 0 0
- joint right_wheel_joint: origin xyz=-0.029784 -1.1174 0 rpy=-1.5708 0 0 -> xyz=-0.029784 -0.76743 0 rpy=-1.5708 0 0
